Commit message: Replace chassis box primitive with accurate shaped STL mesh
Generates chassis.stl from the real acrylic plate outline:
  - Rounded rectangular main body (rear corners R=15mm)
  - Curved front bumper arc (circle C=(25,0)mm, R=85mm)
    fitting the 150mm-wide body at x=65mm to tip at x=110mm
  - Total: 220×150×3mm, origin centered, output in meters

Co-Authored-By: Claude Sonnet 4.6 <noreply@anthropic.com>

File: example/public/robots/robot-car/robot-car.urdf (robot description, URDF)
Before this commit: robot robot-car, 11 links, 10 joints
Links:
- link base_link: geometry visual mesh filename=chassis.stl

Commit message: Orient robot-car so bumper faces viewer by default
The viewer camera sits at Three.js (-1, 0.7, 1) which maps to the -X
side of the URDF frame. Flip chassis STL X axis (bumper now at -X) and
mirror all joint X positions so the bumper is camera-facing and appears
as the prominent front of the robot without needing to rotate the view.

Co-Authored-By: Claude Sonnet 4.6 <noreply@anthropic.com>

File: example/public/robots/robot-car/robot-car.urdf (robot description, URDF)
Before this commit: robot robot-car, 11 links, 10 joints
Joints:
- joint battery_9v_joint: origin xyz=-0.050 -0.038 -0.0135 rpy=0 0 0 -> xyz=0.050 -0.038 -0.0135 rpy=0 0 0
- joint caster_joint: origin xyz=-0.090 0.000 -0.022 rpy=0 0 0 -> xyz=0.090 0.000 -0.022 rpy=0 0 0
- joint esp32cam_joint: origin xyz=0.080 0.000 0.0090 rpy=0 0 0 -> xyz=-0.080 0.000 0.0090 rpy=0 0 0
- joint hcsr04_joint: origin xyz=0.110 0.000 0.0090 rpy=0 0 0 -> xyz=-0.110 0.000 0.0090 rpy=0 0 0
- joint l298n_joint: origin xyz=-0.020 0.042 0.0153 rpy=0 0 0 -> xyz=0.020 0.042 0.0153 rpy=0 0 0
- joint motor_left_joint: origin xyz=0.010 0.040 -0.009 rpy=0 0 0 -> xyz=-0.010 0.040 -0.009 rpy=0 0 0
- joint motor_right_joint: origin xyz=0.010 -0.040 -0.009 rpy=0 0 0 -> xyz=-0.010 -0.040 -0.009 rpy=0 0 0
- joint powerbank_joint: origin xyz=-0.025 -0.030 0.0220 rpy=0 1.5708 0 -> xyz=0.025 -0.030 0.0220 rpy=0 1.5708 0
- joint wheel_left_joint: origin xyz=0.010 0.090 -0.002 rpy=1.5708 0 0 -> xyz=-0.010 0.090 -0.002 rpy=1.5708 0 0
- joint wheel_right_joint: origin xyz=0.010 -0.090 -0.002 rpy=1.5708 0 0 -> xyz=-0.010 -0.090 -0.002 rpy=1.5708 0 0

Commit message: Replace caster ball with proper wheel assembly, move to front
Replaces the tiny sphere with a three-part caster assembly:
  - caster_plate: 36×36×4 mm square mount plate (silver)
  - caster_fork:  8×30×26 mm U-bracket (silver)
  - caster_wheel: ø38×16 mm rubber wheel (black), axis along Y

Moves assembly from rear (+X) to front (-X at x=−65 mm), matching
the chassis image where the caster is on the forward end.

Co-Authored-By: Claude Sonnet 4.6 <noreply@anthropic.com>

File: example/public/robots/robot-car/robot-car.urdf (robot description, URDF)
Before this commit: robot robot-car, 11 links, 10 joints
Links:
- removed link caster_ball
- added link caster_fork; visual box size=0.008 0.030 0.026
- added link caster_plate; visual box size=0.036 0.036 0.004
- added link caster_wheel; visual cylinder length=0.016 radius=0.019
Joints:
- removed joint caster_joint
- added joint caster_fork_joint: type fixed, parent base_link, child caster_fork, origin xyz=-0.065 0.000 -0.019 rpy=0 0 0
- added joint caster_plate_joint: type fixed, parent base_link, child caster_plate, origin xyz=-0.065 0.000 -0.004 rpy=0 0 0
- added joint caster_wheel_joint: type fixed, parent base_link, child caster_wheel, origin xyz=-0.065 0.000 -0.037 rpy=1.5708 0 0

Commit message: Fix left/right wheel and motor labels
With -X as the robot's forward direction, the RHR gives left = -Y
(not +Y). The original positions followed the standard ROS +X-forward
convention by mistake, placing wheel_left at +Y (the physical right).
Swapped Y coordinates for wheel and motor joints and corrected the
coordinate convention comment.

Co-Authored-By: Claude Sonnet 4.6 <noreply@anthropic.com>

File: example/public/robots/robot-car/robot-car.urdf (robot description, URDF)
Before this commit: robot robot-car, 13 links, 12 joints
Joints:
- joint motor_left_joint: origin xyz=-0.010 0.040 -0.009 rpy=0 0 0 -> xyz=-0.010 -0.040 -0.009 rpy=0 0 0
- joint motor_right_joint: origin xyz=-0.010 -0.040 -0.009 rpy=0 0 0 -> xyz=-0.010 0.040 -0.009 rpy=0 0 0
- joint wheel_left_joint: origin xyz=-0.010 0.090 -0.002 rpy=1.5708 0 0 -> xyz=-0.010 -0.090 -0.002 rpy=1.5708 0 0
- joint wheel_right_joint: origin xyz=-0.010 -0.090 -0.002 rpy=1.5708 0 0 -> xyz=-0.010 0.090 -0.002 rpy=1.5708 0 0

Commit message: Fix power bank position: under chassis, spanning Y axis
Moves the power bank from on top (along X) to the underside of the
chassis (along Y), matching the physical build. Also updates color
to blue to match the actual component.

Co-Authored-By: Claude Sonnet 4.6 <noreply@anthropic.com>

File: example/public/robots/robot-car/robot-car.urdf (robot description, URDF)
Before this commit: robot robot-car, 13 links, 12 joints
Joints:
- joint powerbank_joint: origin xyz=0.025 -0.030 0.0220 rpy=0 1.5708 0 -> xyz=0.025 0.000 -0.019 rpy=1.5708 0 0

Commit message: Fix wheel/caster proportions from verified datasheets
Drive wheels (Adafruit #3763):
- Width corrected 25 mm → 15 mm (engineering drawing confirmed)
- Z raised to +11 mm so car sits flat with caster

TT Motor (Adafruit #3777):
- Box corrected to 70×22×22 mm (body runs along X, not Y)
- Y moved to ±70 mm (shaft 8.7 mm from gearbox face)
- Z raised to +11 mm (shaft at wheel center height)

Caster (W420 / Adafruit #3948, both 20 mm height, 15 mm ball):
- Fork resized to 8×16×9 mm (span from plate to ball)
- Ball changed from 38 mm cylinder to 15 mm sphere
- Ball center at Z=−14 mm (chassis_bottom − 20 mm + 7.5 mm)
- Joint changed fixed → continuous (axis Y) so it spins

Co-Authored-By: Claude Sonnet 4.6 <noreply@anthropic.com>

File: example/public/robots/robot-car/robot-car.urdf (robot description, URDF)
Before this commit: robot robot-car, 13 links, 12 joints
Links:
- link caster_fork: geometry visual box size=0.008 0.016 0.009
- link caster_wheel: geometry visual sphere radius=0.0075
- link motor_left: geometry visual box size=0.070 0.022 0.022
- link motor_right: geometry visual box size=0.070 0.022 0.022
- link wheel_left: geometry visual cylinder length=0.015 radius=0.0325
- link wheel_right: geometry visual cylinder length=0.015 radius=0.0325
Joints:
- joint caster_fork_joint: origin xyz=-0.065 0.000 -0.019 rpy=0 0 0 -> xyz=-0.065 0.000 -0.009 rpy=0 0 0
- joint caster_wheel_joint: axis (none) -> 0 1 0; origin xyz=-0.065 0.000 -0.037 rpy=1.5708 0 0 -> xyz=-0.065 0.000 -0.014; type fixed -> continuous
- joint motor_left_joint: origin xyz=-0.010 -0.040 -0.009 rpy=0 0 0 -> xyz=-0.010 -0.070 0.011 rpy=0 0 0
- joint motor_right_joint: origin xyz=-0.010 0.040 -0.009 rpy=0 0 0 -> xyz=-0.010 0.070 0.011 rpy=0 0 0
- joint wheel_left_joint: origin xyz=-0.010 -0.090 -0.002 rpy=1.5708 0 0 -> xyz=-0.010 -0.090 0.011 rpy=1.5708 0 0
- joint wheel_right_joint: origin xyz=-0.010 0.090 -0.002 rpy=1.5708 0 0 -> xyz=-0.010 0.090 0.011 rpy=1.5708 0 0

Commit message: Revert caster to wheel-type, add yellow hubs, HC-SR04 transducers, comparison pieces
Caster:
- Restored fork + cylinder wheel (user confirmed this matches physical robot)
- Correctly sized: ø16 mm wheel so car sits flat (wheel bottom = drive wheel ground)
- Joint is now continuous so it rolls

Drive wheels:
- Width corrected to 26 mm (full wheel incl. hub, matches Adafruit #3763 spec)
- Yellow hub disc added on inboard face (from artifact-experiment reference)

HC-SR04:
- Two white transducer cylinders added to front face (from artifact-experiment)

Floating comparison pieces (Y +220–260 mm, not attached to car):
- alt_caster_ball: ø15 mm sphere (ball caster alternative)
- alt_caster_original: ø38 mm cylinder (original oversized version)
- alt_wheel_plain: 15 mm plain wheel (no hub, tread-width-only alternative)

Co-Authored-By: Claude Sonnet 4.6 <noreply@anthropic.com>

File: example/public/robots/robot-car/robot-car.urdf (robot description, URDF)
Before this commit: robot robot-car, 13 links, 12 joints
Links:
- added link alt_caster_ball; visual sphere radius=0.0075
- added link alt_caster_original; visual cylinder length=0.016 radius=0.019
- added link alt_wheel_plain; visual cylinder length=0.015 radius=0.0325
- link caster_fork: geometry visual box size=0.008 0.016 0.008
- link caster_wheel: geometry visual cylinder length=0.012 radius=0.008
- link hcsr04: geometry visual box size=0.045 0.020 0.015; visual cylinder length=0.010 radius=0.008
- link wheel_left: geometry visual cylinder length=0.0104 radius=0.0195; visual cylinder length=0.026 radius=0.0325
- link wheel_right: geometry visual cylinder length=0.0104 radius=0.0195; visual cylinder length=0.026 radius=0.0325
Joints:
- added joint alt_caster_ball_joint: type fixed, parent base_link, child alt_caster_ball, origin xyz=-0.065 0.220 -0.0135 rpy=0 0 0
- added joint alt_caster_original_joint: type fixed, parent base_link, child alt_caster_original, origin xyz=-0.065 0.260 -0.0135 rpy=1.5708 0 0
- added joint alt_wheel_plain_joint: type fixed, parent base_link, child alt_wheel_plain, origin xyz=-0.010 0.220 0.011 rpy=1.5708 0 0
- joint caster_fork_joint: origin xyz=-0.065 0.000 -0.009 rpy=0 0 0 -> xyz=-0.065 0.000 -0.0095 rpy=0 0 0
- joint caster_wheel_joint: axis 0 1 0 -> 0 0 1; origin xyz=-0.065 0.000 -0.014 -> xyz=-0.065 0.000 -0.0135 rpy=1.5708 0 0

Commit message: Fix yellow hub axis, add catalog items as labeled floating pieces
Yellow hub fix:
- local Y offset mapped to world Z (upward) due to R_x(π/2) joint rotation
- Corrected to local Z: wheel_left xyz="0 0 -0.0078", wheel_right xyz="0 0 0.0078"
- Hub now sits on the inboard face of each wheel

Floating catalog items (not yet installed, hover for labels):
- ir_sensor: MH IR line sensor 32×14×5 mm (Z+80 mm above car)
- logic_converter: 19×14×3 mm PCB for HC-SR04↔ESP32 level shifting
- encoder_disc_left / encoder_disc_right: ø30 mm × 3 mm for wheel odometry

Removed useless alt_caster_* and alt_wheel_* comparison pieces.

Co-Authored-By: Claude Sonnet 4.6 <noreply@anthropic.com>

File: example/public/robots/robot-car/robot-car.urdf (robot description, URDF)
Before this commit: robot robot-car, 16 links, 15 joints
Links:
- removed link alt_caster_ball
- removed link alt_caster_original
- removed link alt_wheel_plain
- added link encoder_disc_left; visual cylinder length=0.003 radius=0.015
- added link encoder_disc_right; visual cylinder length=0.003 radius=0.015
- added link ir_sensor; visual box size=0.032 0.014 0.005
- added link logic_converter; visual box size=0.019 0.014 0.003
Joints:
- removed joint alt_caster_ball_joint
- removed joint alt_caster_original_joint
- removed joint alt_wheel_plain_joint
- added joint encoder_disc_left_joint: type fixed, parent base_link, child encoder_disc_left, origin xyz=0.020 0.000 0.080 rpy=1.5708 0 0
- added joint encoder_disc_right_joint: type fixed, parent base_link, child encoder_disc_right, origin xyz=0.060 0.000 0.080 rpy=1.5708 0 0
- added joint ir_sensor_joint: type fixed, parent base_link, child ir_sensor, origin xyz=-0.060 0.000 0.080 rpy=0 0 0
- added joint logic_converter_joint: type fixed, parent base_link, child logic_converter, origin xyz=-0.020 0.000 0.080 rpy=0 0 0

Commit message: Improve robot-car model and add Inspector with per-axis scale
- Replace wheel cylinder geometry with generated STL (16×4 tread blocks)
- Motors changed to yellow cylinders matching TT motor shape
- Chassis wrapped in chassis_joint so it's Inspector-selectable
- Inspector: replace uniform scale slider with Sx/Sy/Sz per-axis inputs
- Inspector snippet now includes component name prefix for identification
- Add hover labels and click selection for all joints including fixed ones
  (nearestAnyJoint + onHoverAny/onUnhoverAny in URDFDragControls)
- Calibrate caster, wheel, motor, servo stack, battery box, powerbank positions

Co-Authored-By: Claude Sonnet 4.6 <noreply@anthropic.com>

File: example/public/robots/robot-car/robot-car.urdf (robot description, URDF)
Before this commit: robot robot-car, 17 links, 16 joints
Links:
- removed link battery_9v
- removed link encoder_disc_left
- removed link encoder_disc_right
- removed link esp32cam
- removed link ir_sensor
- removed link logic_converter
- added link arduino_r3; visual box size=0.069 0.054 0.011
- added link battery_box; visual box size=0.062 0.052 0.022
- added link chassis; visual mesh filename=chassis.stl scale=1.07 1.00 1.00
- added link ir_receiver; visual box size=0.010 0.010 0.005
- added link sensor_shield; visual box size=0.054 0.054 0.008
- added link servo_bracket; visual box size=0.040 0.040 0.003
- added link servo_motor; visual box size=0.022 0.012 0.022
- link base_link: geometry 
- link caster_wheel: geometry visual cylinder length=0.0145 radius=0.0097
- link motor_left: geometry visual cylinder length=0.070 radius=0.011
- link motor_right: geometry visual cylinder length=0.070 radius=0.011
- link powerbank: geometry visual cylinder length=0.138 radius=0.0096
- link wheel_left: geometry visual cylinder length=0.012 radius=0.022; visual mesh filename=wheel.stl
- link wheel_right: geometry visual cylinder length=0.012 radius=0.022; visual mesh filename=wheel.stl
Joints:
- removed joint battery_9v_joint
- removed joint encoder_disc_left_joint
- removed joint encoder_disc_right_joint
- removed joint esp32cam_joint
- removed joint ir_sensor_joint
- removed joint logic_converter_joint
- added joint arduino_r3_joint: type fixed, parent base_link, child arduino_r3, origin xyz=0.025 0.000 0.007 rpy=0 0 0
- added joint battery_box_joint: type fixed, parent base_link, child battery_box, origin xyz=0.0300 0.0000 -0.0050 rpy=0.0000 0.0000 0.0000
- added joint chassis_joint: type fixed, parent base_link, child chassis, origin xyz=0 0 0 rpy=0 0 0
- added joint ir_receiver_joint: type fixed, parent base_link, child ir_receiver, origin xyz=-0.090 0.030 0.005 rpy=0 0 0
- added joint sensor_shield_joint: type fixed, parent base_link, child sensor_shield, origin xyz=0.025 0.000 0.017 rpy=0 0 0
- added joint servo_bracket_joint: type fixed, parent base_link, child servo_bracket, origin xyz=-0.0900 0.0000 0.0030 rpy=0.0000 0.0000 0.0000
- added joint servo_motor_joint: type fixed, parent base_link, child servo_motor, origin xyz=-0.0900 0.0000 0.0160 rpy=0.0000 0.0000 0.0000
- joint caster_fork_joint: origin xyz=-0.065 0.000 -0.0095 rpy=0 0 0 -> xyz=-0.0900 0.0000 -0.0095 rpy=0 0 0
- joint caster_plate_joint: origin xyz=-0.065 0.000 -0.004 rpy=0 0 0 -> xyz=-0.0900 0.0000 -0.0040 rpy=0 0 0
- joint caster_wheel_joint: origin xyz=-0.065 0.000 -0.0135 rpy=1.5708 0 0 -> xyz=-0.0900 0.0000 -0.0135 rpy=1.5708 0.0000 0.0000
- joint hcsr04_joint: origin xyz=-0.110 0.000 0.0090 rpy=0 0 0 -> xyz=-0.0900 0.0000 0.0340 rpy=0.0000 0.0000 0.0000
- joint motor_left_joint: origin xyz=-0.010 -0.070 0.011 rpy=0 0 0 -> xyz=0.0400 -0.0700 0.0110 rpy=0.0000 0.0000 0.0000
- joint motor_right_joint: origin xyz=-0.010 0.070 0.011 rpy=0 0 0 -> xyz=0.0400 0.0700 0.0110 rpy=0.0000 0.0000 0.0000
- joint powerbank_joint: origin xyz=0.025 0.000 -0.019 rpy=1.5708 0 0 -> xyz=-0.030 0.000 -0.0095 rpy=1.5708 0 0
- joint wheel_left_joint: origin xyz=-0.010 -0.090 0.011 rpy=1.5708 0 0 -> xyz=0.0400 -0.0900 0.0110 rpy=1.5708 0.0000 0.0000
- joint wheel_right_joint: origin xyz=-0.010 0.090 0.011 rpy=1.5708 0 0 -> xyz=0.0400 0.0900 0.0110 rpy=1.5708 0.0000 0.0000

Commit message: Calibrate robot-car component positions and geometry
- Motors and wheels moved below chassis (Z=-0.011)
- Caster assembly re-attached to chassis underside with extended fork
- Chassis narrowed 10% in Y; motors/wheels pulled in proportionally
- Removed servo bracket, HC-SR04, IR receiver, Arduino, sensor shield
- Per-component position/scale tuning: caster wheel, powerbank, battery
  box, L298N (now red)
- Inspector: per-axis scale (Sx/Sy/Sz) replaces uniform slider
- Inspector snippet includes component name prefix

Co-Authored-By: Claude Sonnet 4.6 <noreply@anthropic.com>

File: example/public/robots/robot-car/robot-car.urdf (robot description, URDF)
Before this commit: robot robot-car, 18 links, 17 joints
Links:
- removed link arduino_r3
- removed link hcsr04
- removed link ir_receiver
- removed link sensor_shield
- removed link servo_bracket
- removed link servo_motor
- link battery_box: geometry visual box size=0.0806 0.0442 0.022
- link caster_fork: geometry visual box size=0.008 0.016 0.030
- link caster_wheel: geometry visual cylinder length=0.0145 radius=0.0146
- link chassis: geometry visual mesh filename=chassis.stl scale=1.07 0.90 1.00
- link l298n: geometry visual box size=0.0434 0.0533 0.0055
- link powerbank: geometry visual cylinder length=0.141 radius=0.0115
Joints:
- removed joint arduino_r3_joint
- removed joint hcsr04_joint
- removed joint ir_receiver_joint
- removed joint sensor_shield_joint
- removed joint servo_bracket_joint
- removed joint servo_motor_joint
- joint battery_box_joint: origin xyz=0.0300 0.0000 -0.0050 rpy=0.0000 0.0000 0.0000 -> xyz=0.0460 0.0000 -0.0120 rpy=0.0000 0.0000 0.0000
- joint caster_fork_joint: origin xyz=-0.0900 0.0000 -0.0095 rpy=0 0 0 -> xyz=-0.0900 0.0000 -0.0180 rpy=0.0000 0.0000 0.0000
- joint caster_wheel_joint: origin xyz=-0.0900 0.0000 -0.0135 rpy=1.5708 0.0000 0.0000 -> xyz=-0.0900 0.0000 -0.0320 rpy=1.5708 0.0000 0.0000
- joint l298n_joint: origin xyz=0.020 0.042 0.0153 rpy=0 0 0 -> xyz=0.0500 0.0000 0.0050 rpy=0.0000 0.0000 0.0000
- joint motor_left_joint: origin xyz=0.0400 -0.0700 0.0110 rpy=0.0000 0.0000 0.0000 -> xyz=0.0400 -0.0630 -0.0110 rpy=0.0000 0.0000 0.0000
- joint motor_right_joint: origin xyz=0.0400 0.0700 0.0110 rpy=0.0000 0.0000 0.0000 -> xyz=0.0400 0.0630 -0.0110 rpy=0.0000 0.0000 0.0000
- joint powerbank_joint: origin xyz=-0.030 0.000 -0.0095 rpy=1.5708 0 0 -> xyz=-0.0300 0.0000 -0.0110 rpy=1.5708 0.0000 0.0000
- joint wheel_left_joint: origin xyz=0.0400 -0.0900 0.0110 rpy=1.5708 0.0000 0.0000 -> xyz=0.0400 -0.0810 -0.0110 rpy=1.5708 0.0000 0.0000
- joint wheel_right_joint: origin xyz=0.0400 0.0900 0.0110 rpy=1.5708 0.0000 0.0000 -> xyz=0.0400 0.0810 -0.0110 rpy=1.5708 0.0000 0.0000

Commit message: Move motors inward 6 mm and add sidebar pin option
- Shift motor_left Y from -0.063 → -0.057, motor_right symmetrically to +0.057
- Add 📌 pin button to sidebar header; when active, backdrop click no longer closes the panel
- Update CLAUDE.md motor positions table to match current URDF

Co-Authored-By: Claude Sonnet 4.6 <noreply@anthropic.com>

File: example/public/robots/robot-car/robot-car.urdf (robot description, URDF)
Before this commit: robot robot-car, 12 links, 11 joints
Joints:
- joint motor_left_joint: origin xyz=0.0400 -0.0630 -0.0110 rpy=0.0000 0.0000 0.0000 -> xyz=0.0400 -0.0570 -0.0110 rpy=0.0000 0.0000 0.0000
- joint motor_right_joint: origin xyz=0.0400 0.0630 -0.0110 rpy=0.0000 0.0000 0.0000 -> xyz=0.0400 0.0570 -0.0110 rpy=0.0000 0.0000 0.0000
