Commit message: update

File: docs/robots/robot-car/robot-car.urdf (robot description, URDF)
Before this commit: robot robot-car, 12 links, 11 joints
Joints:
- joint caster_fork_joint: origin xyz=-0.0900 0.0000 -0.0180 rpy=0.0000 0.0000 0.0000 -> xyz=-0.1300 0.0000 -0.0180 rpy=0.0000 0.0000 0.0000
- joint caster_plate_joint: origin xyz=-0.0900 0.0000 -0.0040 rpy=0 0 0 -> xyz=-0.1300 0.0000 -0.0040 rpy=0 0 0
- joint caster_wheel_joint: origin xyz=-0.0900 0.0000 -0.0320 rpy=1.5708 0.0000 0.0000 -> xyz=-0.1300 0.0000 -0.0320 rpy=1.5708 0.0000 0.0000
