Commit message: Update robot-car caster and powerbank positions; document parts-based URDF assembly
- Caster assembly (plate/fork/wheel): X −0.090 → −0.130 m
- Powerbank: X −0.030 → −0.093 m, length 0.141 → 0.1199 m
- CLAUDE.md: document that robot-car.urdf is assembled from parts/ on every build

Co-Authored-By: Claude Sonnet 4.6 <noreply@anthropic.com>

File: docs/robots/robot-car/robot-car.urdf (robot description, URDF)
Before this commit: robot robot-car, 12 links, 11 joints
Links:
- link motor_left: geometry visual mesh filename=tt_can.stl; visual mesh filename=tt_gearbox.stl
- link motor_right: geometry visual mesh filename=tt_can.stl; visual mesh filename=tt_gearbox.stl
- link powerbank: geometry visual cylinder length=0.1199 radius=0.0115

Commit message: robot-car: replace motor cylinders with STL meshes; fix caster and powerbank positions
- Motors now use tt_gearbox.stl, tt_can.stl, tt_shaft.stl instead of cylinders
- Caster assembly moved from X=-0.090 to X=-0.130
- Powerbank length corrected (141→120 mm) and position moved to X=-0.093
- Add gen_chassis.cjs, gen_motor.cjs generator scripts to docs
- Rebuild docs assets

Co-Authored-By: Claude Sonnet 4.6 <noreply@anthropic.com>

File: docs/robots/robot-car/robot-car.urdf (robot description, URDF)
Before this commit: robot robot-car, 12 links, 11 joints
Joints:
- joint powerbank_joint: origin xyz=-0.0300 0.0000 -0.0110 rpy=1.5708 0.0000 0.0000 -> xyz=-0.0930 0.0000 -0.0110 rpy=1.5708 0.0000 0.0000
